File: hardware/prj-kicad/mcu.kicad_sch (KiCad schematic)
At the start: 10 parts, among them U1 ATSAMC21J

Commit message: Hardware: Finish current sensor interface and create production files for rev1
Parts:
- added TP7, TP8: CONN_1, cowdin-3a-pwrmon:TP_2SMD, symbol cowdin-3a-pwrmon:CONN_1
Connections:
- net CT4_I: now reaches U1.13 (PA04)
- net CT1_OUT: now reaches U1.15 (PA06)
- net at U1.17 (PA08): now also TP7.1
- net at U1.18 (PA09): now also TP8.1
- net CT2_OUT: now reaches U1.5 (PB04)
- net RELAY: now reaches U1.63 (PB02)
- net CT_SEL1: now reaches U1.64 (PB03)
- no-connect marks 4 -> 8
Changed lines of the file:
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@@
   (no_connect (at 100.965 86.36))
   (no_connect (at 100.965 88.9))
+  (no_connect (at 73.025 71.12))
   (no_connect (at 187.96 82.55))
   (no_connect (at 187.96 85.09))
+  (no_connect (at 73.025 76.2))
+  (no_connect (at 73.025 83.82))
+  (no_connect (at 73.025 86.36))
   (wire (pts (xy 83.185 104.14) (xy 83.185 105.41))
     (stroke (width 0) (type default) (color 0 0 0 0))
   )
+  (wire (pts (xy 152.4 74.93) (xy 154.94 74.93))
+    (stroke (width 0) (type default) (color 0 0 0 0))
+  )
   (wire (pts (xy 81.28 159.385) (xy 81.28 160.655))
     (stroke (width 0) (type default) (color 0 0 0 0))
@@
     (stroke (width 0) (type default) (color 0 0 0 0))
   )
+  (wire (pts (xy 70.485 81.28) (xy 73.025 81.28))
+    (stroke (width 0) (type default) (color 0 0 0 0))
+  )
   (wire (pts (xy 168.91 52.07) (xy 168.91 50.8))
     (stroke (width 0) (type default) (color 0 0 0 0))
@@
     (stroke (width 0) (type default) (color 0 0 0 0))
   )
+  (wire (pts (xy 152.4 72.39) (xy 154.94 72.39))
+    (stroke (width 0) (type default) (color 0 0 0 0))
+  )
   (wire (pts (xy 191.77 52.07) (xy 191.77 49.53))
     (stroke (width 0) (type default) (color 0 0 0 0))
@@
     (stroke (width 0) (type default) (color 0 0 0 0))
   )
+  (wire (pts (xy 70.485 68.58) (xy 73.025 68.58))
+    (stroke (width 0) (type default) (color 0 0 0 0))
+  )
   (wire (pts (xy 171.45 50.8) (xy 171.45 52.07))
     (stroke (width 0) (type default) (color 0 0 0 0))
@@
     (stroke (width 0) (type default) (color 0 0 0 0))
   )
+  (wire (pts (xy 70.485 78.74) (xy 73.025 78.74))
+    (stroke (width 0) (type default) (color 0 0 0 0))
+  )
   (wire (pts (xy 129.54 146.685) (xy 129.54 147.955))
     (stroke (width 0) (type default) (color 0 0 0 0))
   )
+  (wire (pts (xy 152.4 69.85) (xy 154.94 69.85))
+    (stroke (width 0) (type default) (color 0 0 0 0))
+  )
+  (wire (pts (xy 70.485 73.66) (xy 73.025 73.66))
+    (stroke (width 0) (type default) (color 0 0 0 0))
+  )
   (wire (pts (xy 100.965 60.96) (xy 103.505 60.96))
     (stroke (width 0) (type default) (color 0 0 0 0))
@@
     )
   )
+  (global_label "CT2_OUT" (shape input) (at 152.4 74.93 180) (fields_autoplaced)
+    (effects (font (size 1.016 1.016)) (justify right))
+    (property "Intersheet References" "${INTERSHEET_REFS}" (id 0) (at 144.0349 74.8665 0)
+      (effects (font (size 1.016 1.016)) (justify right) hide)
+    )
+  )
   (global_label "RS485_TX" (shape output) (at 70.485 88.9 180) (fields_autoplaced)
     (effects (font (size 1.016 1.016)) (justify right))
@@
     )
   )
+  (global_label "CT4_I" (shape input) (at 70.485 68.58 180) (fields_autoplaced)
+    (effects (font (size 1.016 1.016)) (justify right))
+    (property "Intersheet References" "${INTERSHEET_REFS}" (id 0) (at 64.539 68.5165 0)
+      (effects (font (size 1.016 1.016)) (justify right) hide)
+    )
+  )
   (global_label "SWDAT" (shape bidirectional) (at 103.505 96.52 0) (fields_autoplaced)
     (effects (font (size 1.016 1.016)) (justify left))
@@
     )
   )
+  (global_label "RELAY" (shape output) (at 152.4 69.85 180) (fields_autoplaced)
+    (effects (font (size 1.016 1.016)) (justify right))
+    (property "Intersheet References" "${INTERSHEET_REFS}" (id 0) (at 145.9702 69.7865 0)
+      (effects (font (size 1.016 1.016)) (justify right) hide)
+    )
+  )
   (global_label "RS485_DIR" (shape output) (at 70.485 93.98 180) (fields_autoplaced)
     (effects (font (size 1.016 1.016)) (justify right))
@@
     )
   )
+  (global_label "CT_SEL1" (shape output) (at 152.4 72.39 180) (fields_autoplaced)
+    (effects (font (size 1.016 1.016)) (justify right))
+    (property "Intersheet References" "${INTERSHEET_REFS}" (id 0) (at 144.2285 72.3265 0)
+      (effects (font (size 1.016 1.016)) (justify right) hide)
+    )
+  )
   (global_label "EXT_RX" (shape input) (at 189.865 67.31 0) (fields_autoplaced)
     (effects (font (size 1.016 1.016)) (justify left))
@@
     (property "Intersheet References" "${INTERSHEET_REFS}" (id 0) (at 139.3081 147.8915 0)
       (effects (font (size 1.016 1.016)) (justify left) hide)
+    )
+  )
+  (global_label "CT1_OUT" (shape input) (at 70.485 73.66 180) (fields_autoplaced)
+    (effects (font (size 1.016 1.016)) (justify right))
+    (property "Intersheet References" "${INTERSHEET_REFS}" (id 0) (at 62.1199 73.5965 0)
+      (effects (font (size 1.016 1.016)) (justify right) hide)
     )
   )
@@
     (pin "2")
   )
+  (symbol (lib_id "cowdin-3a-pwrmon:CONN_1") (at 66.675 81.28 180) (unit 1)
+    (in_bom yes) (on_board yes)
+    (property "Reference" "TP8" (id 0) (at 65.405 81.28 0)
+      (effects (font (size 1.016 1.016)) (justify left))
+    )
+    (property "Value" "CONN_1" (id 1) (at 66.675 82.677 0)
+      (effects (font (size 0.762 0.762)) hide)
+    )
+    (property "Footprint" "cowdin-3a-pwrmon:TP_2SMD" (id 2) (at 66.675 81.28 0)
+      (effects (font (size 1.524 1.524)) hide)
+    )
+    (property "Datasheet" "" (id 3) (at 66.675 81.28 0)
+      (effects (font (size 1.524 1.524)))
+    )
+    (pin "1")
+  )
   (symbol (lib_id "cowdin-3a-pwrmon:GND") (at 171.45 101.6 0) (unit 1)
     (in_bom yes) (on_board yes) (fields_autoplaced)
@@
       (effects (font (size 1.524 1.524)))
     )
+    (pin "1")
+  )
+  (symbol (lib_id "cowdin-3a-pwrmon:CONN_1") (at 66.675 78.74 180) (unit 1)
+    (in_bom yes) (on_board yes)
+    (property "Reference" "TP7" (id 0) (at 65.405 78.74 0)
+      (effects (font (size 1.016 1.016)) (justify left))
+    )
+    (property "Value" "CONN_1" (id 1) (at 66.675 80.137 0)
+      (effects (font (size 0.762 0.762)) hide)
+    )
+    (property "Footprint" "cowdin-3a-pwrmon:TP_2SMD" (id 2) (at 66.675 78.74 0)
+      (effects (font (size 1.524 1.524)) hide)
+    )
+    (property "Datasheet" "" (id 3) (at 66.675 78.74 0)
+      (effects (font (size 1.524 1.524)))
+    )
